File: src/qei_board/interface.brd (EAGLE design)
At the start: 160 x 100 mm, 1 part, among them IC1 74LS33N

Commit message: up
Parts:
- added SV1: (no value), con-lstb:MA04-1
Connections:
- new net N$1: IC1.1, SV1.1
- new net N$2: IC1.10, SV1.3
- new net N$3: IC1.4, SV1.2
- new net N$4: IC1.2
- new net N$5: IC1.5
- new net N$6: IC1.9
Changed lines of the file:
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@@
 <elements>
 <element name="IC1" library="74xx-us" package="DIL14" value="74LS33N" x="44.45" y="46.99" rot="R270"/>
+<element name="SV1" library="con-lstb" package="MA04-1" value="" x="11.43" y="-7.62">
+<attribute name="OC_NEWARK" value="unknown" x="11.43" y="-7.62" size="1.778" layer="27" display="off"/>
+<attribute name="MF" value="" x="11.43" y="-7.62" size="1.778" layer="27" display="off"/>
+<attribute name="OC_FARNELL" value="unknown" x="11.43" y="-7.62" size="1.778" layer="27" display="off"/>
+<attribute name="MPN" value="" x="11.43" y="-7.62" size="1.778" layer="27" display="off"/>
+</element>
 </elements>
 <signals>
@@
 <contactref element="IC1" pad="14"/>
 </signal>
+<signal name="N$1">
+<contactref element="IC1" pad="1"/>
+<contactref element="SV1" pad="1"/>
+<wire x1="7.62" y1="-7.62" x2="40.64" y2="54.61" width="0" layer="19" extent="1-1"/>
+</signal>
+<signal name="N$2">
+<contactref element="IC1" pad="10"/>
+<contactref element="SV1" pad="3"/>
+<wire x1="12.7" y1="-7.62" x2="48.26" y2="44.45" width="0" layer="19" extent="1-1"/>
+</signal>
+<signal name="N$3">
+<contactref element="IC1" pad="4"/>
+<contactref element="SV1" pad="2"/>
+<wire x1="10.16" y1="-7.62" x2="40.64" y2="46.99" width="0" layer="19" extent="1-1"/>
+</signal>
+<signal name="N$4">
+<contactref element="IC1" pad="2"/>
+</signal>
+<signal name="N$5">
+<contactref element="IC1" pad="5"/>
+</signal>
+<signal name="N$6">
+<contactref element="IC1" pad="9"/>
+</signal>
 </signals>
