File: src/qei_board/interface.sch (EAGLE design)
At the start: 1 part, among them IC1 74LS33N

Commit message: up
Parts:
- added SV1: (no value), con-lstb:MA04-1
Connections:
- new net N$1: IC1A.O, SV1.1
- new net N$2: IC1C.O, SV1.3
- new net N$3: IC1B.O, SV1.2
- new net N$4: IC1A.I0
- new net N$5: IC1B.I0
- new net N$6: IC1C.I1
Other:
- note added: "HOME1"
- note added: "INDX1"
- note added: "QEIB1_IN"
- note added: "RPA14"
- note added: "RPB6"
- note added: "RPB9"
Changed lines of the file:
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@@
 <parts>
 <part name="IC1" library="74xx-us" deviceset="74*33" device="N" technology="LS"/>
+<part name="SV1" library="con-lstb" deviceset="MA04-1" device=""/>
 </parts>
 <sheets>
 <sheet>
 <plain>
+<text x="27.94" y="76.2" size="1.778" layer="91">RPA14</text>
+<text x="25.4" y="40.64" size="1.778" layer="91">RPB6</text>
+<text x="22.86" y="73.66" size="1.778" layer="91">QEIB1_IN</text>
+<text x="25.4" y="38.1" size="1.778" layer="91">INDX1</text>
+<text x="20.32" y="55.88" size="1.778" layer="91">HOME1</text>
+<text x="25.4" y="58.42" size="1.778" layer="91">RPB9</text>
 </plain>
 <instances>
@@
 <instance part="IC1" gate="C" x="10.16" y="40.64"/>
 <instance part="IC1" gate="D" x="10.16" y="20.32"/>
+<instance part="SV1" gate="1" x="48.26" y="50.8" rot="R180"/>
 </instances>
 <busses>
 </busses>
 <nets>
+<net name="N$1" class="0">
+<segment>
+<pinref part="IC1" gate="A" pin="O"/>
+<wire x1="22.86" y1="76.2" x2="35.56" y2="76.2" width="0.1524" layer="91"/>
+<wire x1="35.56" y1="76.2" x2="35.56" y2="55.88" width="0.1524" layer="91"/>
+<pinref part="SV1" gate="1" pin="1"/>
+<wire x1="35.56" y1="55.88" x2="40.64" y2="55.88" width="0.1524" layer="91"/>
+</segment>
+</net>
+<net name="N$2" class="0">
+<segment>
+<pinref part="IC1" gate="C" pin="O"/>
+<wire x1="22.86" y1="40.64" x2="35.56" y2="40.64" width="0.1524" layer="91"/>
+<wire x1="35.56" y1="40.64" x2="35.56" y2="50.8" width="0.1524" layer="91"/>
+<pinref part="SV1" gate="1" pin="3"/>
+<wire x1="35.56" y1="50.8" x2="40.64" y2="50.8" width="0.1524" layer="91"/>
+</segment>
+</net>
+<net name="N$3" class="0">
+<segment>
+<pinref part="IC1" gate="B" pin="O"/>
+<wire x1="22.86" y1="58.42" x2="30.48" y2="58.42" width="0.1524" layer="91"/>
+<wire x1="30.48" y1="58.42" x2="30.48" y2="53.34" width="0.1524" layer="91"/>
+<pinref part="SV1" gate="1" pin="2"/>
+<wire x1="30.48" y1="53.34" x2="40.64" y2="53.34" width="0.1524" layer="91"/>
+</segment>
+</net>
+<net name="N$4" class="0">
+<segment>
+<pinref part="IC1" gate="A" pin="I0"/>
+<wire x1="-2.54" y1="78.74" x2="-30.48" y2="78.74" width="0.1524" layer="91"/>
+<wire x1="-30.48" y1="78.74" x2="-30.48" y2="81.28" width="0.1524" layer="91"/>
+</segment>
+</net>
+<net name="N$5" class="0">
+<segment>
+<pinref part="IC1" gate="B" pin="I0"/>
+<wire x1="-2.54" y1="60.96" x2="-30.48" y2="60.96" width="0.1524" layer="91"/>
+</segment>
+</net>
+<net name="N$6" class="0">
+<segment>
+<pinref part="IC1" gate="C" pin="I1"/>
+<wire x1="-2.54" y1="38.1" x2="-30.48" y2="38.1" width="0.1524" layer="91"/>
+<wire x1="-30.48" y1="38.1" x2="-30.48" y2="40.64" width="0.1524" layer="91"/>
+</segment>
+</net>
 </nets>
 </sheet>
